File: walter-feels/kicadproject/sensors.kicad_sch (KiCad schematic)
At the start: 11 parts, among them Q5 DMP2021UFDE-7, U10 SCD30, U7 HDC1080DMBR, U8 BMP280, U9 LSM6DSM

Commit message: Updated Walter schematic to v1.5 and updated Walter Feels to version 2.1
Parts:
- removed U8: BMP280, Package_LGA:Bosch_LGA-8_2x2.5mm_P0.65mm_ClockwisePinNumbering, symbol Sensor_Pressure:BMP280
- added U8: LPS22HBTR, LPS22HBTR:HLGA10_2X2_STM-L, symbol LPS22HBTR:LPS22HBTR
Connections:
- net 3V3: now also U8.1 (VDD_IO), U8.10 (VDD), U8.6 (CS)
- net GND: now also U8.3 (RES), U8.5 (SDO/SA0), U8.8 (GND), U8.9 (GND)
- net I2C_SCL: now also U8.2 (SCL/SPC)
- net I2C_SDA: now also U8.4 (SDA/SDI/SDO)
- no-connect marks 6 -> 7
Other:
- moved on the sheet: C48, C49

Commit message: Updated Walter Feels to V2.3
Parts:
- U8: JLCPCB (none) -> C94049
Changed lines of the file:
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@@
   (title_block
     (title "Walter Feels")
-    (date "2023-10-13")
-    (rev "2.1")
+    (date "2024-03-13")
+    (rev "2.3")
     (company "DPTechnics BV")
     (comment 1 "Checked by: Jonas Maes")
@@
       (effects (font (size 1.27 1.27) italic) hide)
     )
+    (property "JLCPCB" "C94049" (id 4) (at 95.885 93.345 0)
+      (effects (font (size 1.27 1.27)) hide)
+    )
     (pin "1")

Commit message: Updated Walter Feels project to version 2.6
Changed lines of the file:
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@@
   (title_block
     (title "Walter Feels")
-    (date "2025-02-12")
-    (rev "2.4")
+    (date "2026-01-13")
+    (rev "2.6")
     (company "DPTechnics BV")
     (comment 1 "Checked by: Jonas Maes")
@@
   )
   (symbol (lib_id "SCD30:SCD30") (at 240.665 115.57 0) (mirror x) (unit 1)
-    (in_bom yes) (on_board yes) (fields_autoplaced)
-    (property "Reference" "U10" (id 0) (at 254.635 92.71 0))
-    (property "Value" "SCD30" (id 1) (at 254.635 95.25 0))
+    (in_bom yes) (on_board yes)
+    (property "Reference" "U10" (id 0) (at 254.635 93.98 0))
+    (property "Value" "SCD30" (id 1) (at 254.635 96.52 0))
     (property "Footprint" "SCD30:SCD30" (id 2) (at 240.665 115.57 0)
       (effects (font (size 1.27 1.27)) hide)
