File: walter-feels/kicadproject/walter-feels.kicad_sch (KiCad schematic)
At the start: 17 parts, among them J2 1071010, J3 1071010, J4 1990070, J5 1990070, U1 DPT_Walter

Commit message: Updated Walter Feels to V2.3
Parts:
- removed FID1, FID2, FID3, FID4: Fiducial, Fiducial:Fiducial_0.5mm_Mask1mm, symbol Mechanical:Fiducial
- removed H1, H2, H3, H4: MountingHole, MountingHole:MountingHole_2.7mm_M2.5_ISO14580, symbol Mechanical:MountingHole
- added F1: 5A Slow, Fuse:Fuse_1206_3216Metric, symbol Device:Fuse
- added J6: Conn_01x04_Male, Connector_PinHeader_2.54mm:PinHeader_1x04_P2.54mm_Vertical, symbol Connector:Conn_01x04_Male
- J2, J3: JLCPCB (none) -> C3310307
- J4, J5: JLCPCB (none) -> C17275119
Connections:
- net RS485_RX_EN is gone; now on net RS485_TX_EN: U1.22 (IO18)
- net +3.3V: now also J6.1 (Pin_1)
- net 12V_EN: now also U1.3 (TX0/IO43); no longer U1.4 (IO0/~{3V3-EN})
- net GND: now also J6.4 (Pin_4)
- net I2C_SCL: now also J6.2 (Pin_2)
- net I2C_SDA: now also J6.3 (Pin_3)
- net RS232_TX_EN: now also U1.21 (IO17); no longer U1.20 (IO16)
- net RS485_TX_EN: no longer U1.21 (IO17)
- net SDI12_RX_EN: now also U1.24 (IO9); no longer U1.23 (IO8)
- net SDI12_TX_EN: now also U1.25 (IO10); no longer U1.24 (IO9)
- net VBAT: now also F1.2; no longer J3.2
- net ~{RS232_RX_EN}: now also U1.20 (IO16); no longer U1.19 (IO15)
- net ~{CAN_EN}: now reaches U1.2 (RX0/IO44)
- net 1W_3V3_IO renamed CAN_RX
- net 1W_DAT renamed CAN_L
- net 1W_GND renamed CAN_H
- net CO2_EN renamed ~{CO2_EN}
- new net: F1.1, J3.2
- new net CAN_TX: U1.19 (IO15)
- new net ~{RS485_RX_EN}: U1.23 (IO8)
- no-connect marks 3 -> 2
Other:
- sheet Serial ports ports: added CAN_H, CAN_L, CAN_RX, CAN_TX, SDI12_RX_EN, ~{CAN_EN}; removed 1W_3V3_IO, 1W_DAT, 1W_GND, ~{SDI12_RX_EN}
- moved on the sheet: J2, J3, J4, J5

Commit message: Updated Walter Feels project to version 2.6
Parts:
- added C34, C35: 10nF, Capacitor_SMD:C_0603_1608Metric, symbol Device:C
- added D4, D5: 8.2V, Diode_SMD:D_SOD-523, symbol Device:D_Zener
- added F2: 5A Slow, Fuse:Fuse_1206_3216Metric, symbol Device:Fuse
- added Q4, Q6: CSD17318Q2, footprints:CSD17318Q2, symbol symbols:CSD17318Q2
- added R16, R17, R18: 8.2MΩ, Resistor_SMD:R_0603_1608Metric, symbol Device:R
Connections:
- net +3.3V: now also R16.1
- net GND: now also Q4.1, Q6.1; no longer J2.2, J3.1
- net I2C_BUSPOW: now also R1.2, R2.2; no longer R1.1, R2.1
- net I2C_SCL: now also R1.1; no longer R1.2
- net I2C_SDA: now also R2.1; no longer R2.2
- net VBAT: now also F2.2, R18.2; no longer F1.2
- net VSOLAR: now also F1.2, R17.2; no longer J2.1
- net at F1.1: now also J2.1; no longer J3.2
- net SYSPOWER_GOOD: now reaches U1.1 (~{RESET})
- net at U1.4 (IO0/~{3V3-EN}): now also R16.2
- new net: C35.1, D5.1 (K), Q4.3, R18.1
- new net: C35.2, D5.2 (A), J3.1, Q4.2
- new net: C34.2, D4.2 (A), J2.2, Q6.2
- new net: C34.1, D4.1 (K), Q6.3, R17.1
- new net: F2.1, J3.2
- no-connect marks 2 -> 0
Other:
- sheet Power ports: added SYSPOWER_GOOD; removed none
- moved on the sheet: J2, J4, J5, J6, R1, R2
